File: Assembly/PCB/Layout.sch (KiCad schematic (older format))
At the start: 192 parts, among them SW1 SW_1U, SW10 SW_1U, SW11 SW_1U, SW12 SW_1U, SW13 SW_1U, SW14 SW_1U, SW15 SW_1U, SW16 SW_1U, SW17 SW_1U, SW18 SW_1U, SW19 SW_1U, SW2 SW_1U, SW20 SW_1U, SW21 SW_1U, SW22 SW_1U, SW23 SW_1U, SW24 SW_1U, SW25 SW_1U, SW26 SW_1U, SW27 SW_1U, SW28 SW_1U, SW29 SW_1U, SW3 SW_1U, SW30 SW_2U, SW31 SW_1U, SW32 SW_1.5U, SW33 SW_1U, SW34 SW_1U, SW35 SW_1U, SW36 SW_1U, SW37 SW_1U, SW38 SW_1U, SW39 SW_1U, SW4 SW_1U, SW40 SW_1U, SW41 SW_1U, SW42 SW_1U, SW43 SW_1U, SW44 SW_1U, SW45 SW_ENTER_ANSIISO, SW46 SW_1U, SW47 SW_1.75U, SW48 SW_1U, SW49 SW_1U, SW5 SW_1U, SW50 SW_1U, SW51 SW_1U, SW52 SW_1U, SW53 SW_1U, SW54 SW_1U, SW55 SW_1U, SW56 SW_1U, SW57 SW_1U, SW58 SW_1U, SW59 SW_PIPE_ANSIISO, SW6 SW_1U, SW60 SW_1U, SW61 SW_LSHIFT_ANSIISO, SW62 SW_1U, SW63 SW_1U, SW64 SW_1U, SW65 SW_1U, SW66 SW_1U, SW67 SW_1U, SW68 SW_1U, SW69 SW_1U, SW7 SW_1U, SW70 SW_1U, SW71 SW_1U, SW72 SW_1U, SW73 SW_1.75U, SW74 SW_1U, SW75 SW_1U, SW76 SW_1.25, SW77 SW_1.25, SW78 SW_1.25, SW79 SW_6.25U, SW8 SW_1U, SW80 SW_1U, SW81 SW_1U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

Commit message: Added descriptors for BOM generation
Parts:
- D1, D10, D11, D12, D13, D14, D15, D16, D17, D18, D19, D2, D20, D21, D22, D23, D24, D25, D26, D27, D28, D29, D3, D30, D31, D32, D33, D34, D35, D36, D37, D38, D39, D4, D40, D41, D42, D43, D44, D45, D46, D47, D48, D49, D5, D50, D51, D52, D53, D54, D55, D56, D57, D58, D59, D6, D60, D61, D62, D63, D64, D65, D66, D67, D68, D69, D7, D70, D71, D72, D73, D74, D75, D76, D77, D78, D79, D8, D80, D81, D82, D83, D84, D85, D9: value D -> 1N4148; Description (none) -> 75V +150℃@(Tj) 200mW Single 1.25V@150mA 4ns 1μA@75V 150mA S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; ExtPrice (none) -> 0.64; LCSC C448648 -> C129870; Link (none) -> https://lcsc.com/product-detail/Switching-Diode_DIYI-Elec-T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; Manufaturer (none) -> DIYI Elec Tech; MfgPart (none) -> 1N4148WS-HE3-18; Minimum (none) -> 50; Multiples (none) -> 50; Package (none) -> SOD-323; Type (none) -> SMD
- SW1, SW10, SW11, SW12, SW13, SW14, SW15, SW16, SW17, SW18, SW19, SW2, SW20, SW21, SW22, SW23, SW24, SW25, SW26, SW27, SW28, SW29, SW3, SW30, SW31, SW32, SW33, SW34, SW35, SW36, SW37, SW38, SW39, SW4, SW40, SW41, SW42, SW43, SW44, SW45, SW46, SW47, SW48, SW49, SW5, SW50, SW51, SW52, SW53, SW54, SW55, SW56, SW57, SW58, SW59, SW6, SW60, SW61, SW62, SW63, SW64, SW65, SW66, SW67, SW68, SW69, SW7, SW70, SW71, SW72, SW73, SW74, SW75, SW76, SW77, SW78, SW79, SW8, SW80, SW81, SW82, SW83, SW84, SW85, SW9: Package (none) -> CherryMx; Population (none) -> DNP; Type (none) -> thru-hole
- TP1, TP10, TP11, TP12, TP13, TP14, TP15, TP16, TP17, TP18, TP19, TP2, TP20, TP21, TP22, TP3, TP4, TP5, TP6, TP7, TP8, TP9: Description (none) -> -; LCSC (none) -> -; Link (none) -> -; Manufaturer (none) -> -; MfgPart (none) -> -; Minimum (none) -> -; Multiples (none) -> -; Package (none) -> -; Population (none) -> DNP; Type (none) -> -
