File: Assembly/PCB/PCB.sch (KiCad schematic (older format))
At the start: 35 parts, among them P1 USB_C_Plug_USB2.0, U1 ATmega32U4-MU, Y1 16MHz

Commit message: Added descriptors for BOM generation
Parts:
- C1, C2, C3, C4, C5, C6: Description (none) -> 16V 100nF X5R ±10% 0402 Multilayer Ceramic Capacitors MLCC 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; ExtPrice (none) -> 0.10; Link (none) -> https://lcsc.com/product-detail/Multilayer-Ceramic-Capacito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; Manufaturer (none) -> YAGEO; MfgPart (none) -> CC0402KRX5R7BB104; Minimum (none) -> 100; Multiples (none) -> 100; Package (none) -> 0402; Type (none) -> SMD; Unit Price (none) -> 0.0010
- C7: Description (none) -> 50V 22pF C0G ±5% 0402 Multilayer Ceramic Capacitors MLCC - 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; ExtPrice (none) -> 0.11; Link (none) -> https://lcsc.com/product-detail/Multilayer-Ceramic-Capacito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; Manufaturer (none) -> FH(Guangdong Fenghua Advanced Tech); MfgPart (none) -> 0402CG220J500NT; Minimum (none) -> 100; Multiples (none) -> 100; Package (none) -> 0402; Type (none) -> SMD; Unit Price (none) -> 0.0011
- C8: value 22pf -> 22pF; Description (none) -> 50V 22pF C0G ±5% 0402 Multilayer Ceramic Capacitors MLCC - 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; ExtPrice (none) -> 0.11; Link (none) -> https://lcsc.com/product-detail/Multilayer-Ceramic-Capacito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; Manufaturer (none) -> FH(Guangdong Fenghua Advanced Tech); MfgPart (none) -> 0402CG220J500NT; Minimum (none) -> 100; Multiples (none) -> 100; Package (none) -> 0402; Type (none) -> SMD; Unit Price (none) -> 0.0011
- C9: Description (none) -> 16V 1uF X5R ±10% 0402 Multilayer Ceramic Capacitors MLCC - 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; ExtPrice (none) -> 0.26; Link (none) -> https://lcsc.com/product-detail/Multilayer-Ceramic-Capacito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; Manufaturer (none) -> Taiyo Yuden; MfgPart (none) -> EMK105BJ105KV-F; Minimum (none) -> 50; Multiples (none) -> 50; Package (none) -> 0402; Type (none) -> SMD; Unit Price (none) -> 0.0052
- FID1, FID2, FID3, FID4, H1, H10, H11, H2, H3, H4, H5, H6, H7, H8, H9, JP1: Description (none) -> -; LCSC (none) -> -; Link (none) -> -; Manufaturer (none) -> -; MfgPart (none) -> -; Minimum (none) -> -; Multiples (none) -> -; Package (none) -> -; Population (none) -> DNP; Type (none) -> -; Unit Price (none) -> -
- P1: Description (none) -> 1 Surface Mount 16 Female Type-C SMD USB Connectors ROHS; ExtPrice (none) -> 0.57; Link (none) -> https://lcsc.com/product-detail/USB-Connectors_HCTL-HC-TYPE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; Manufaturer (none) -> HCTL; MfgPart (none) -> HC-TYPE-C-16P-01B; Minimum (none) -> 5; Multiples (none) -> 5; Package (none) -> SMD; Type (none) -> SMD
- R1, R2, R3, R4: Description (none) -> ±1% 1/16W Thick Film Resistors 50V ±100ppm/℃ -55℃~+155℃ 5.1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; ExtPrice (none) -> 0.07; Link (none) -> https://lcsc.com/product-detail/Chip-Resistor-Surface-Mount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; Manufaturer (none) -> UNI-ROYAL(Uniroyal Elec); MfgPart (none) -> 0402WGF5101TCE; Minimum (none) -> 100; Multiples (none) -> 100; Package (none) -> 0402; Type (none) -> SMD
- R5: Description (none) -> ±5% 1/16W Thick Film Resistors 50V ±100ppm/℃ -55℃~+155℃ 300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; ExtPrice (none) -> 0.07; Link (none) -> https://lcsc.com/product-detail/Chip-Resistor-Surface-Mount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; Manufaturer (none) -> UNI-ROYAL(Uniroyal Elec); MfgPart (none) -> 0402WGJ0301TCE; Minimum (none) -> 100; Multiples (none) -> 100; Package (none) -> 0402; Type (none) -> SMD
- TP23, TP24: Description (none) -> -; LCSC (none) -> -; Link (none) -> -; Manufaturer (none) -> -; MfgPart (none) -> -; Minimum (none) -> -; Multiples (none) -> -; Package (none) -> -; Population (none) -> DNP; Type (none) -> -
- U1: Description (none) -> 16MHz AVR 2.7V ~ 5.5V QFN-44_7x7x05P ATMEL & AVR ROHS; ExtPrice (none) -> 9.36; LCSC (none) -> C112161; Link (none) -> https://lcsc.com/product-detail/ATMEL-AVR_Microchip-Tech-AT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; Manufaturer (none) -> Microchip Tech; MfgPart (none) -> ATMEGA32U4-MU; Minimum (none) -> 1; Multiples (none) -> 1; Package (none) -> QFN-44_7x7x05P; Type (none) -> SMD
- Y1: Description (none) -> 16MHz SMD Crystal Resonator 9pF ±10ppm ±30ppm -40℃~+85℃ SMD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; ExtPrice (none) -> 0.44; Link (none) -> https://lcsc.com/product-detail/Crystals_Yangxing-Tech-X322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; Manufaturer (none) -> Yangxing Tech; MfgPart (none) -> X322516MLB4SI; Minimum (none) -> 5; Multiples (none) -> 5; Package (none) -> SMD3225-4P; Type (none) -> SMD
