File: Assembly/PCB/rgb.sch (KiCad schematic (older format))
At the start: 176 parts

Commit message: Added descriptors for BOM generation
Parts:
- C10, C11, C12, C13, C14, C15, C16, C17, C18, C19, C20, C21, C22, C23, C24, C25, C26, C27, C28, C29, C30, C31, C32, C33, C34, C35, C36, C37, C38, C39, C40, C41, C42, C43, C44, C45, C46, C47, C48, C49, C50, C51, C52, C53, C54, C55, C56, C57, C58, C59, C60, C61, C62, C63, C64, C65, C66, C67, C68, C69, C70, C71, C72, C73, C74, C75, C76, C77, C78, C79, C80, C81, C82, C83, C84, C85, C86, C87, C88, C89, C90, C91, C92, C93, C94, C95, C96, C97: Description (none) -> 16V 100nF X5R ±10% 0402 Multilayer Ceramic Capacitors MLCC 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; ExtPrice (none) -> 0.10; Link (none) -> https://lcsc.com/product-detail/Multilayer-Ceramic-Capacito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; Manufaturer (none) -> YAGEO; MfgPart (none) -> CC0402KRX5R7BB104; Minimum (none) -> 100; Multiples (none) -> 100; Package (none) -> 0402; Type (none) -> SMD; Unit Price (none) -> 0.0010
- D100, D101, D102, D103, D104, D105, D106, D107, D108, D109, D110, D111, D112, D113, D114, D115, D116, D117, D118, D119, D120, D121, D122, D123, D124, D125, D126, D127, D128, D129, D130, D131, D132, D133, D134, D135, D136, D137, D138, D139, D140, D141, D142, D143, D144, D145, D146, D147, D148, D149, D150, D151, D152, D153, D154, D155, D156, D157, D158, D159, D160, D161, D162, D163, D164, D165, D166, D167, D168, D169, D170, D171, D172, D173, D86, D87, D88, D89, D90, D91, D92, D93, D94, D95, D96, D97, D98, D99: Type (none) -> SMD

Commit message: Added Component_BOM
Parts:
- D100, D101, D102, D103, D104, D105, D106, D107, D108, D109, D110, D111, D112, D113, D114, D115, D116, D117, D118, D119, D120, D121, D122, D123, D124, D125, D126, D127, D128, D129, D130, D131, D132, D133, D134, D135, D136, D137, D138, D139, D140, D141, D142, D143, D144, D145, D146, D147, D148, D149, D150, D151, D152, D153, D154, D155, D156, D157, D158, D159, D160, D161, D162, D163, D164, D165, D166, D167, D168, D169, D170, D171, D172, D173, D86, D87, D88, D89, D90, D91, D92, D93, D94, D95, D96, D97, D98, D99: ExtPrice (none) -> 10.40; Link (none) -> https://es.aliexpress.com/item/4000475685852.html?spm=a2g0o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; Minimum (none) -> 100; Multiples (none) -> 100
